Commit message: Add topic prefix && Test gr2t5

File: assets/urdf/GR1T1.urdf (robot description, URDF)
Before this commit: robot GR1T1, 37 links, 36 joints
Links:
- link IMU_link: geometry visual mesh filename=../meshes/gr1t1/IMU_link.STL
- link base_link: geometry collision cylinder length=0.1371007021179978 radius=0.12239433188500067; visual mesh filename=../meshes/gr1t1/base_link.STL
- link head_pitch_link: geometry collision sphere radius=0.1086868692306477; visual mesh filename=../meshes/gr1t1/head_pitch_link.STL
- link head_roll_link: geometry visual mesh filename=../meshes/gr1t1/head_roll_link.STL
- link head_yaw_link: geometry visual mesh filename=../meshes/gr1t1/head_yaw_link.STL
- link left_foot_pitch_link: geometry visual mesh filename=../meshes/gr1t1/left_foot_pitch_link.STL
- link left_foot_roll_link: geometry collision cylinder length=0.24 radius=0.02; collision cylinder length=0.24 radius=0.02
- link left_hand_pitch_link: geometry visual mesh filename=../meshes/gr1t1/left_hand_pitch_link.STL
- link left_hand_roll_link: geometry visual mesh filename=../meshes/gr1t1/left_hand_roll_link.STL
- link left_hand_yaw_link: geometry collision cylinder length=0.1391873595177893 radius=0.04157192402358859; visual mesh filename=../meshes/gr1t1/left_hand_yaw_link.STL
- link left_lower_arm_pitch_link: geometry visual mesh filename=../meshes/gr1t1/left_lower_arm_pitch_link.STL
- link left_shank_pitch_link: geometry collision cylinder length=0.18076995129198576 radius=0.05332138187428352; visual mesh filename=../meshes/gr1t1/left_shank_pitch_link.STL
- link left_thigh_pitch_link: geometry collision cylinder length=0.24982894507630515 radius=0.08587689590118133; visual mesh filename=../meshes/gr1t1/left_thigh_pitch_link.STL
- link left_thigh_roll_link: geometry visual mesh filename=../meshes/gr1t1/left_thigh_roll_link.STL
- link left_thigh_yaw_link: geometry visual mesh filename=../meshes/gr1t1/left_thigh_yaw_link.STL
- link left_upper_arm_pitch_link: geometry visual mesh filename=../meshes/gr1t1/left_upper_arm_pitch_link.STL
- link left_upper_arm_roll_link: geometry visual mesh filename=../meshes/gr1t1/left_upper_arm_roll_link.STL
- link left_upper_arm_yaw_link: geometry collision cylinder length=0.1698839909625244 radius=0.03623321337242011; visual mesh filename=../meshes/gr1t1/left_upper_arm_yaw_link.STL
- link right_foot_pitch_link: geometry visual mesh filename=../meshes/gr1t1/right_foot_pitch_link.STL
- link right_foot_roll_link: geometry collision cylinder length=0.24 radius=0.02; collision cylinder length=0.24 radius=0.02
- link right_hand_pitch_link: geometry visual mesh filename=../meshes/gr1t1/right_hand_pitch_link.STL
- link right_hand_roll_link: geometry visual mesh filename=../meshes/gr1t1/right_hand_roll_link.STL
- link right_hand_yaw_link: geometry collision cylinder length=0.1391873595177893 radius=0.04157192402358859; visual mesh filename=../meshes/gr1t1/right_hand_yaw_link.STL
- link right_lower_arm_pitch_link: geometry visual mesh filename=../meshes/gr1t1/right_lower_arm_pitch_link.STL
- link right_shank_pitch_link: geometry collision cylinder length=0.180768239886 radius=0.053321055277056; visual mesh filename=../meshes/gr1t1/right_shank_pitch_link.STL
- link right_thigh_pitch_link: geometry collision cylinder length=0.24982123520352716 radius=0.0858779947877418; visual mesh filename=../meshes/gr1t1/right_thigh_pitch_link.STL
- link right_thigh_roll_link: geometry visual mesh filename=../meshes/gr1t1/right_thigh_roll_link.STL
- link right_thigh_yaw_link: geometry visual mesh filename=../meshes/gr1t1/right_thigh_yaw_link.STL
- link right_upper_arm_pitch_link: geometry visual mesh filename=../meshes/gr1t1/right_upper_arm_pitch_link.STL
- link right_upper_arm_roll_link: geometry visual mesh filename=../meshes/gr1t1/right_upper_arm_roll_link.STL
- link right_upper_arm_yaw_link: geometry collision cylinder length=0.1698839909625244 radius=0.03623321337242011; visual mesh filename=../meshes/gr1t1/right_upper_arm_yaw_link.STL
- link torso_link: geometry collision cylinder length=0.1603859984881334 radius=0.12742740516179015; visual mesh filename=../meshes/gr1t1/torso_link.STL
- link waist_pitch_link: geometry visual mesh filename=../meshes/gr1t1/waist_pitch_link.STL
- link waist_roll_link: geometry visual mesh filename=../meshes/gr1t1/waist_roll_link.STL
- link waist_yaw_link: geometry visual mesh filename=../meshes/gr1t1/waist_yaw_link.STL
